File: Hardware/nucular-keyboard.sch (KiCad schematic (older format))
At the start: 34 parts, among them IC1 STM32L052R6Tx, J1 JAE-AA01B-S040VA1, J2 JAE-KX14-K2D, J3 CONN_01X16, J4 CONN_01X03, Q1 IRLML6402, U1 MCP1700T-3302E/MB

Commit message: Big clean-up
Parts:
- removed D1: PRTR5V0U2X, TO_SOT_Packages_SMD:SOT-143B_reflow, symbol PRTR5V0U2X
- removed J1: JAE-AA01B-S040VA1, Connectors_JAE:JAE_AA01B-S040VA1_2x20x0.5mm, symbol JAE-AA01B-S040VA1
- removed J2: JAE-KX14-K2D, Connectors_JAE:JAE_KX14-K2D_2x20x0.8mm, symbol JAE-KX14-KxD
- removed U1: MCP1700T-3302E/MB, TO_SOT_Packages_SMD:SOT89-3_Housing, symbol MCP1700T-3302E/MB
- added D1: PRTR5V0U2X, _TkModules:SOT143B, symbol Nexperia_PRTR5V0U2X
- added J1: JAE_AA01B-S040VA1, _TkModules:JAE_AA01B-S040VA1, symbol JAE_AA01B-S040VA1
- added J2: JAE_KX14-40K2D, _TkModules:JAE_KX14-40K2D, symbol JAE_KX14-40K2D
- added U1: MCP1700T-3302E/MB, _TkModules:SOT89-3, symbol Microchip_MCP1700T-3302E/MB
- USB1: value USB_OTG -> Molex_105017-0001; footprint Connectors_USB:USB_Micro-B_Molex-105017-0001 -> _TkModules:Molex_105017-0001_USB-Micro-B
Changed lines of the file:
@@
 LIBS:valves
 LIBS:stm32
-LIBS:MCP1700T-3302E-MB
 LIBS:nxp
 LIBS:ir
-LIBS:nucular-keyboard-cache
+LIBS:_TkComponents
 EELAYER 26 0
 EELAYER END
@@
 Text Label 11950 2850 0    60   ~ 0
 PWRSWITCH
-$Comp
-L JAE-AA01B-S040VA1 J1
-U 1 1 58F660DD
-P 11100 2850
-F 0 "J1" H 11100 4237 60  0000 C CNN
-F 1 "JAE-AA01B-S040VA1" H 11100 4131 60  0000 C CNN
-F 2 "Connectors_JAE:JAE_AA01B-S040VA1_2x20x0.5mm" H 10350 2950 60  0001 C CNN
-F 3 "" H 10350 2950 60  0001 C CNN
-	1    11100 2850
-	1    0    0    -1
-$EndComp
-$Comp
-L JAE-KX14-KxD J2
-U 1 1 58F660DE
-P 14150 2850
-F 0 "J2" H 14150 4187 60  0000 C CNN
-F 1 "JAE-KX14-K2D" H 14150 4081 60  0000 C CNN
-F 2 "Connectors_JAE:JAE_KX14-K2D_2x20x0.8mm" H 14150 2750 60  0001 C CNN
-F 3 "" H 14150 2750 60  0001 C CNN
-	1    14150 2850
-	1    0    0    -1
-$EndComp
 Text Label 11950 3750 0    60   ~ 0
 TP4_DATA
@@
 $EndComp
 $Comp
-L MCP1700T-3302E/MB U1
-U 1 1 58F668D4
-P 3800 9400
-F 0 "U1" H 3800 9767 50  0000 C CNN
-F 1 "MCP1700T-3302E/MB" H 3800 9676 50  0000 C CNN
-F 2 "TO_SOT_Packages_SMD:SOT89-3_Housing" H 3800 9500 50  0001 C CNN
-F 3 "" H 3800 9500 50  0001 C CNN
-	1    3800 9400
-	1    0    0    -1
-$EndComp
-$Comp
 L USB_OTG USB1
 U 1 1 58F668D5
 P 1700 7700
 F 0 "USB1" H 1755 8167 50  0000 C CNN
-F 1 "USB_OTG" H 1755 8076 50  0000 C CNN
-F 2 "Connectors_USB:USB_Micro-B_Molex-105017-0001" H 1850 7650 50  0001 C CNN
+F 1 "Molex_105017-0001" H 1755 8076 50  0000 C CNN
+F 2 "_TkModules:Molex_105017-0001_USB-Micro-B" H 1850 7650 50  0001 C CNN
 F 3 "" H 1850 7650 50  0001 C CNN
 	1    1700 7700
@@
 	5150 5950 5550 5950
 Wire Wire Line
-	5550 5750 5550 6100
+	5550 5750 5550 6150
 Wire Wire Line
 	5350 5750 5350 5950
@@
 L GND #PWR021
 U 1 1 58FD8629
-P 5550 6100
-F 0 "#PWR021" H 5550 5850 50  0001 C CNN
-F 1 "GND" V 5555 5972 50  0000 R CNN
-F 2 "" H 5550 6100 50  0001 C CNN
-F 3 "" H 5550 6100 50  0001 C CNN
-	1    5550 6100
+P 5550 6150
+F 0 "#PWR021" H 5550 5900 50  0001 C CNN
+F 1 "GND" V 5555 6022 50  0000 R CNN
+F 2 "" H 5550 6150 50  0001 C CNN
+F 3 "" H 5550 6150 50  0001 C CNN
+	1    5550 6150
 	1    0    0    -1
 $EndComp
@@
 	1    10550 4400
 	1    0    0    -1
-$EndComp
-$Comp
-L PRTR5V0U2X D1
-U 1 1 58FE14C8
-P 3800 8350
-F 0 "D1" H 3800 7863 60  0000 C CNN
-F 1 "PRTR5V0U2X" H 3800 7969 60  0000 C CNN
-F 2 "TO_SOT_Packages_SMD:SOT-143B_reflow" H 3700 8600 60  0001 C CNN
-F 3 "" H 3700 8600 60  0001 C CNN
-	1    3800 8350
-	-1   0    0    1
 $EndComp
 Connection ~ 4300 7700
@@
 	0    1    -1   0
 $EndComp
+$Comp
+L Nexperia_PRTR5V0U2X D1
+U 1 1 59092074
+P 3800 8350
+F 0 "D1" H 3800 7863 60  0000 C CNN
+F 1 "PRTR5V0U2X" H 3800 7969 60  0000 C CNN
+F 2 "_TkModules:SOT143B" H 3700 8600 60  0001 C CNN
+F 3 "" H 3700 8600 60  0001 C CNN
+	1    3800 8350
+	-1   0    0    1
+$EndComp
+$Comp
+L JAE_KX14-40K2D J2
+U 1 1 59093E51
+P 14150 2850
+F 0 "J2" H 14200 4237 60  0000 C CNN
+F 1 "JAE_KX14-40K2D" H 14200 4131 60  0000 C CNN
+F 2 "_TkModules:JAE_KX14-40K2D" H 14850 1400 60  0001 C CNN
+F 3 "" H 14200 2750 60  0001 C CNN
+	1    14150 2850
+	1    0    0    -1
+$EndComp
+$Comp
+L Microchip_MCP1700T-3302E/MB U1
+U 1 1 59096F70
+P 3800 9400
+F 0 "U1" H 3800 9767 50  0000 C CNN
+F 1 "MCP1700T-3302E/MB" H 3800 9676 50  0000 C CNN
+F 2 "_TkModules:SOT89-3" H 3800 9050 50  0001 C CNN
+F 3 "" H 3800 9500 50  0001 C CNN
+	1    3800 9400
+	1    0    0    -1
+$EndComp
+$Comp
+L JAE_AA01B-S040VA1 J1
+U 1 1 59093D6D
+P 11100 2850
+F 0 "J1" H 11150 4237 60  0000 C CNN
+F 1 "JAE_AA01B-S040VA1" H 11150 4131 60  0000 C CNN
+F 2 "_TkModules:JAE_AA01B-S040VA1" H 11800 1400 60  0001 C CNN
+F 3 "" H 10400 2900 60  0001 C CNN
+	1    11100 2850
+	1    0    0    -1
+$EndComp
 $EndSCHEMATC

Commit message: Renamed libray to 000-xxx, so it's always on top
Parts:
- D1: footprint _TkModules:SOT143B -> 000-Modules:SOT143B
- J1: footprint _TkModules:JAE_AA01B-S040VA1 -> 000-Modules:JAE_AA01B-S040VA1
- J2: footprint _TkModules:JAE_KX14-40K2D -> 000-Modules:JAE_KX14-40K2D
- U1: footprint _TkModules:SOT89-3 -> 000-Modules:SOT89-3
- USB1: footprint _TkModules:Molex_105017-0001_USB-Micro-B -> 000-Modules:Molex_105017-0001_USB-Micro-B
Changed lines of the file:
@@
 LIBS:nxp
 LIBS:ir
-LIBS:_TkComponents
+LIBS:000-Components
 EELAYER 26 0
 EELAYER END
@@
 F 0 "USB1" H 1755 8167 50  0000 C CNN
 F 1 "Molex_105017-0001" H 1755 8076 50  0000 C CNN
-F 2 "_TkModules:Molex_105017-0001_USB-Micro-B" H 1850 7650 50  0001 C CNN
+F 2 "000-Modules:Molex_105017-0001_USB-Micro-B" H 1850 7650 50  0001 C CNN
 F 3 "" H 1850 7650 50  0001 C CNN
 	1    1700 7700
@@
 F 0 "D1" H 3800 7863 60  0000 C CNN
 F 1 "PRTR5V0U2X" H 3800 7969 60  0000 C CNN
-F 2 "_TkModules:SOT143B" H 3700 8600 60  0001 C CNN
+F 2 "000-Modules:SOT143B" H 3700 8600 60  0001 C CNN
 F 3 "" H 3700 8600 60  0001 C CNN
 	1    3800 8350
@@
 F 0 "J2" H 14200 4237 60  0000 C CNN
 F 1 "JAE_KX14-40K2D" H 14200 4131 60  0000 C CNN
-F 2 "_TkModules:JAE_KX14-40K2D" H 14850 1400 60  0001 C CNN
+F 2 "000-Modules:JAE_KX14-40K2D" H 14850 1400 60  0001 C CNN
 F 3 "" H 14200 2750 60  0001 C CNN
 	1    14150 2850
@@
 F 0 "U1" H 3800 9767 50  0000 C CNN
 F 1 "MCP1700T-3302E/MB" H 3800 9676 50  0000 C CNN
-F 2 "_TkModules:SOT89-3" H 3800 9050 50  0001 C CNN
+F 2 "000-Modules:SOT89-3" H 3800 9050 50  0001 C CNN
 F 3 "" H 3800 9500 50  0001 C CNN
 	1    3800 9400
@@
 F 0 "J1" H 11150 4237 60  0000 C CNN
 F 1 "JAE_AA01B-S040VA1" H 11150 4131 60  0000 C CNN
-F 2 "_TkModules:JAE_AA01B-S040VA1" H 11800 1400 60  0001 C CNN
+F 2 "000-Modules:JAE_AA01B-S040VA1" H 11800 1400 60  0001 C CNN
 F 3 "" H 10400 2900 60  0001 C CNN
 	1    11100 2850

Commit message: fill polys
Connections:
- net GND: now also J4.2 (P2); no longer J4.1 (P1)
- net SWCLK: now also J4.3 (P3); no longer J4.2 (P2)
- net SWDIO: now also J4.1 (P1); no longer J4.3 (P3)
Changed lines of the file:
@@
 LIBS:ir
 LIBS:000-Components
+LIBS:nucular-keyboard-cache
 EELAYER 26 0
 EELAYER END
@@
 L GND #PWR07
 U 1 1 58F65977
-P 10800 7650
-F 0 "#PWR07" H 10800 7400 50  0001 C CNN
-F 1 "GND" V 10805 7522 50  0000 R CNN
-F 2 "" H 10800 7650 50  0001 C CNN
-F 3 "" H 10800 7650 50  0001 C CNN
-	1    10800 7650
+P 10750 7750
+F 0 "#PWR07" H 10750 7500 50  0001 C CNN
+F 1 "GND" V 10755 7622 50  0000 R CNN
+F 2 "" H 10750 7750 50  0001 C CNN
+F 3 "" H 10750 7750 50  0001 C CNN
+	1    10750 7750
 	0    1    1    0
 $EndComp
@@
 Text Label 1200 2150 2    60   ~ 0
 /RESET
+Text Label 11100 7650 2    60   ~ 0
+SWDIO
 Text Label 11100 7850 2    60   ~ 0
-SWDIO
-Text Label 11100 7750 2    60   ~ 0
 SWCLK
 $Comp
@@
 	11250 6200 11100 6200
 Wire Wire Line
-	11250 7650 10800 7650
-Wire Wire Line
-	11250 7750 11100 7750
+	11250 7650 11100 7650
+Wire Wire Line
+	11250 7750 10750 7750
 Wire Wire Line
 	11250 7850 11100 7850
